File: project4_mcu_datalogger.kicad_sch (KiCad schematic)
At the start: 25 parts, among them U1 24LC1025, U2 24LC1025, U3 ATMEGA328P-AU, U4 DS1337S_T_R, Y1 32.768 KHz, Y2 16 MHz

Commit message: Completed placement of footprints
Parts:
- renumbered U4 to U2, U2 to U3, U3 to U4
Changed lines of the file:
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@@
 		(dnp no)
 		(fields_autoplaced yes)
-		(property "Reference" "U4"
+		(property "Reference" "U2"
 			(at 57.15 36.83 0)
 			(effects
@@
 			(project ""
 				(path "/6791cede-e2c8-424a-b751-f1a182bcbb22"
-					(reference "U4")
+					(reference "U2")
 					(unit 1)
 				)
@@
 		(on_board yes)
 		(dnp no)
-		(property "Reference" "U2"
+		(property "Reference" "U3"
 			(at 71.12 129.54 0)
 			(effects
@@
 			(project "project4_mcu_datalogger"
 				(path "/6791cede-e2c8-424a-b751-f1a182bcbb22"
-					(reference "U2")
+					(reference "U3")
 					(unit 1)
 				)
@@
 		(dnp no)
 		(fields_autoplaced yes)
-		(property "Reference" "U3"
+		(property "Reference" "U4"
 			(at 217.17 33.02 0)
 			(effects
@@
 			(project ""
 				(path "/6791cede-e2c8-424a-b751-f1a182bcbb22"
-					(reference "U3")
-					(unit 1)
-				)
+					(reference "U4")
+					(unit 1)
+				)

Commit message: Completed PCB routing
Parts:
- renumbered C3 to C2, C2 to C3
Changed lines of the file:
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@@
 		(dnp no)
 		(fields_autoplaced yes)
-		(property "Reference" "C2"
+		(property "Reference" "C3"
 			(at 152.4 68.58 90)
 			(effects
@@
 			(project "project4_mcu_datalogger"
 				(path "/6791cede-e2c8-424a-b751-f1a182bcbb22"
-					(reference "C2")
+					(reference "C3")
 					(unit 1)
 				)
@@
 		(dnp no)
 		(fields_autoplaced yes)
-		(property "Reference" "C3"
+		(property "Reference" "C2"
 			(at 152.4 55.88 90)
 			(effects
@@
 			(project "project4_mcu_datalogger"
 				(path "/6791cede-e2c8-424a-b751-f1a182bcbb22"
-					(reference "C3")
-					(unit 1)
-				)
+					(reference "C2")
+					(unit 1)
+				)

Commit message: Fixed outstanding issues
Connections:
- net Vcc: now also BT1.1 (+), C5.1, D2.2 (A), U4.18 (AVCC), U4.6 (VCC__1)
Changed lines of the file:
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@@
+		)
+	)
+	(label "Vcc"
+		(at 266.7 40.64 0)
+		(effects
+			(font
+				(size 1.27 1.27)
+			)
+			(justify left bottom)
 		)
 	)

Commit message: Fixed two defects in the schematic
Connections:
- net SCK: no longer R3.2, U1.6 (SCL), U2.6 (SCL), U3.6 (SCL), U4.28 (PC5)
- new net SCL: R3.2, U1.6 (SCL), U2.6 (SCL), U3.6 (SCL), U4.28 (PC5)
Other:
- sheet Connectors ports: added SCL; removed none
Changed lines of the file:
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@@
 	(wire
 		(pts
-			(xy 181.61 152.4) (xy 187.96 152.4)
-		)
-		(stroke
-			(width 0)
-			(type default)
-		)
-	)
-	(wire
-		(pts
 			(xy 64.77 143.51) (xy 64.77 151.13)
 		)
@@
 	(wire
 		(pts
-			(xy 187.96 139.7) (xy 181.61 139.7)
+			(xy 21.59 52.07) (xy 39.37 52.07)
 		)
 		(stroke
@@
 	(wire
 		(pts
-			(xy 21.59 52.07) (xy 39.37 52.07)
+			(xy 187.96 60.96) (xy 201.93 60.96)
 		)
 		(stroke
@@
 	(wire
 		(pts
-			(xy 187.96 60.96) (xy 201.93 60.96)
+			(xy 74.93 36.83) (xy 88.9 36.83)
 		)
 		(stroke
@@
 	(wire
 		(pts
-			(xy 74.93 36.83) (xy 88.9 36.83)
+			(xy 232.41 45.72) (xy 237.49 45.72)
 		)
 		(stroke
@@
 	(wire
 		(pts
-			(xy 232.41 45.72) (xy 237.49 45.72)
+			(xy 187.96 50.8) (xy 187.96 60.96)
 		)
 		(stroke
@@
 	(wire
 		(pts
-			(xy 187.96 50.8) (xy 187.96 60.96)
+			(xy 170.18 76.2) (xy 186.69 76.2)
 		)
 		(stroke
@@
 	(wire
 		(pts
-			(xy 170.18 76.2) (xy 186.69 76.2)
+			(xy 181.61 151.13) (xy 187.96 151.13)
 		)
 		(stroke
@@
 	(wire
 		(pts
+			(xy 181.61 140.97) (xy 187.96 140.97)
+		)
+		(stroke
+			(width 0)
+			(type default)
+		)
+	)
+	(wire
+		(pts
 			(xy 255.27 40.64) (xy 269.24 40.64)
 		)
@@
 	(wire
 		(pts
+			(xy 181.61 148.59) (xy 187.96 148.59)
+		)
+		(stroke
+			(width 0)
+			(type default)
+		)
+	)
+	(wire
+		(pts
 			(xy 99.06 151.13) (xy 82.55 151.13)
 		)
@@
 	(wire
 		(pts
-			(xy 246.38 82.55) (xy 246.38 95.25)
+			(xy 181.61 138.43) (xy 187.96 138.43)
 		)
 		(stroke
@@
 	(wire
 		(pts
-			(xy 246.38 67.31) (xy 246.38 74.93)
+			(xy 246.38 82.55) (xy 246.38 95.25)
 		)
 		(stroke
@@
 	(wire
 		(pts
-			(xy 170.18 127) (xy 187.96 127)
+			(xy 246.38 67.31) (xy 246.38 74.93)
 		)
 		(stroke
@@
 	(wire
 		(pts
-			(xy 109.22 36.83) (xy 115.57 36.83)
+			(xy 170.18 127) (xy 187.96 127)
 		)
 		(stroke
@@
 	(wire
 		(pts
-			(xy 238.76 99.06) (xy 238.76 101.6)
+			(xy 109.22 36.83) (xy 115.57 36.83)
 		)
 		(stroke
@@
 	(wire
 		(pts
-			(xy 187.96 147.32) (xy 181.61 147.32)
+			(xy 238.76 99.06) (xy 238.76 101.6)
 		)
 		(stroke
@@
 	(wire
 		(pts
-			(xy 21.59 60.96) (xy 21.59 62.23)
+			(xy 181.61 144.78) (xy 187.96 144.78)
 		)
 		(stroke
@@
 	(wire
 		(pts
-			(xy 166.37 36.83) (xy 134.62 36.83)
+			(xy 21.59 60.96) (xy 21.59 62.23)
 		)
 		(stroke
@@
 	(wire
 		(pts
-			(xy 187.96 142.24) (xy 181.61 142.24)
+			(xy 166.37 36.83) (xy 134.62 36.83)
 		)
 		(stroke
@@
 	(wire
 		(pts
-			(xy 246.38 35.56) (xy 246.38 40.64)
-		)
-		(stroke
-			(width 0)
-			(type default)
-		)
-	)
-	(wire
-		(pts
 			(xy 115.57 52.07) (xy 115.57 73.66)
 		)
@@
 	(wire
 		(pts
-			(xy 74.93 67.31) (xy 80.01 67.31)
+			(xy 181.61 153.67) (xy 187.96 153.67)
 		)
 		(stroke
@@
 	(wire
 		(pts
-			(xy 99.06 143.51) (xy 99.06 151.13)
+			(xy 74.93 67.31) (xy 80.01 67.31)
 		)
 		(stroke
@@
 	(wire
 		(pts
-			(xy 134.62 36.83) (xy 134.62 50.8)
+			(xy 99.06 143.51) (xy 99.06 151.13)
 		)
 		(stroke
@@
 	(wire
 		(pts
-			(xy 148.59 50.8) (xy 134.62 50.8)
+			(xy 134.62 36.83) (xy 134.62 50.8)
 		)
 		(stroke
@@
 	(wire
 		(pts
-			(xy 175.26 50.8) (xy 187.96 50.8)
+			(xy 148.59 50.8) (xy 134.62 50.8)
 		)
 		(stroke
@@
 	(wire
 		(pts
-			(xy 187.96 149.86) (xy 181.61 149.86)
+			(xy 175.26 50.8) (xy 187.96 50.8)
 		)
 		(stroke
@@
 		)
 	)
-	(label "SCK"
+	(label "SCL"
 		(at 92.71 140.97 0)
 		(effects
@@
 	)
 	(label "RESET"
-		(at 181.61 152.4 180)
+		(at 181.61 153.67 180)
 		(effects
 			(font
@@
 		)
 	)
-	(label "SCK"
+	(label "SCL"
 		(at 110.49 149.86 180)
 		(effects
@@
 		)
 	)
-	(label "SCK"
+	(label "SCL"
 		(at 59.69 140.97 0)
 		(effects
@@
 		)
 	)
-	(label "SCK"
+	(label "SCL"
 		(at 201.93 83.82 180)
 		(effects
@@
 	)
 	(label "TX"
-		(at 181.61 139.7 180)
+		(at 181.61 138.43 180)
 		(effects
 			(font
@@
 		)
 	)
-	(label "SCK"
+	(label "SCL"
 		(at 39.37 49.53 180)
 		(effects
@@
 	)
 	(label "RX"
-		(at 181.61 142.24 180)
+		(at 181.61 140.97 180)
 		(effects
 			(font
@@
 		)
 	)
+	(label "SCL"
+		(at 181.61 144.78 180)
+		(effects
+			(font
+				(size 1.27 1.27)
+			)
+			(justify right bottom)
+		)
+	)
 	(label "MISO"
-		(at 181.61 149.86 180)
+		(at 181.61 151.13 180)
 		(effects
 			(font
@@
 	)
 	(label "MOSI"
-		(at 181.61 147.32 180)
+		(at 181.61 148.59 180)
 		(effects
 			(font
@@
 	)
 	(symbol
-		(lib_id "power:PWR_FLAG")
-		(at 246.38 35.56 0)
-		(unit 1)
-		(exclude_from_sim no)
-		(in_bom yes)
-		(on_board yes)
-		(dnp no)
-		(fields_autoplaced yes)
-		(property "Reference" "#FLG01"
-			(at 246.38 33.655 0)
-			(effects
-				(font
-					(size 1.27 1.27)
-				)
-				(hide yes)
-			)
-		)
-		(property "Value" "PWR_FLAG"
-			(at 246.38 30.48 0)
-			(effects
-				(font
-					(size 1.27 1.27)
-				)
-			)
-		)
-		(property "Footprint" ""
-			(at 246.38 35.56 0)
-			(effects
-				(font
-					(size 1.27 1.27)
-				)
-				(hide yes)
-			)
-		)
-		(property "Datasheet" "~"
-			(at 246.38 35.56 0)
-			(effects
-				(font
-					(size 1.27 1.27)
-				)
-				(hide yes)
-			)
-		)
-		(property "Description" "Special symbol for telling ERC where power comes from"
-			(at 246.38 35.56 0)
-			(effects
-				(font
-					(size 1.27 1.27)
-				)
-				(hide yes)
-			)
-		)
-		(pin "1"
-		)
-		(instances
-			(project "project4_mcu_datalogger"
-				(path "/6791cede-e2c8-424a-b751-f1a182bcbb22"
-					(reference "#FLG01")
-					(unit 1)
-				)
-			)
-		)
-	)
-	(symbol
 		(lib_id "Device:LED")
 		(at 171.45 50.8 0)
@@
 	(sheet
 		(at 187.96 120.65)
-		(size 16.51 34.925)
+		(size 16.51 35.56)
 		(exclude_from_sim no)
 		(in_bom yes)
@@
 		)
 		(property "Sheetfile" "connectors.kicad_sch"
-			(at 187.96 156.1596 0)
+			(at 187.96 157.48 0)
 			(effects
 				(font
@@
 		)
 		(pin "RESET" passive
-			(at 187.96 152.4 180)
+			(at 187.96 153.67 180)
 			(effects
 				(font
@@
 		)
 		(pin "TX" output
-			(at 187.96 139.7 180)
+			(at 187.96 138.43 180)
 			(effects
 				(font
@@
 		)
 		(pin "MISO" output
-			(at 187.96 149.86 180)
+			(at 187.96 151.13 180)
 			(effects
 				(font
@@
 		)
 		(pin "MOSI" input
-			(at 187.96 147.32 180)
+			(at 187.96 148.59 180)
 			(effects
 				(font
@@
 		)
 		(pin "RX" input
-			(at 187.96 142.24 180)
+			(at 187.96 140.97 180)
+			(effects
+				(font
+					(size 1.27 1.27)
+				)
+				(justify left)
+			)
+		)
+		(pin "SCL" passive
+			(at 187.96 144.78 180)
 			(effects
 				(font
